Commit message: add 3-D intersection experiment setup, while the scale is still an issue

File: src/od_description/urdf/racecar.xacro (robot description, xacro)
@@ -252,5 +252,5 @@
   </link>
   <joint name="mono_camera_joint" type="fixed">
-    <origin xyz="0.390 0 0.01" rpy="0 0 0"/>
+    <origin xyz="0.390 0 0.5" rpy="0 0 0"/>
     <axis xyz="0 0 1" />
     <parent link="chassis"/>
